File: schematic/main_v1.kicad_sch (KiCad schematic)
At the start: 12 parts

Commit message: Created revision 1.1 of main_v1
Parts:
- removed U?: RTL-SDR, symbol payload_symbol_library:RTL-SDR
- removed U?: BBB_Wireless, symbol payload_symbol_library:BBB_Wireless
- added U5: BBB_Wireless_Reduced, symbol payload_symbol_library:BBB_Wireless_Reduced
- gave numbers to parts that had none: 10
Connections:
- net GND: now reaches C2. (-), C3.2, M2.3 (-), U1. (Vout), U2. (Vs)
- net GND: now also BT1.2 (-), C1. (-); no longer U3. (Vin), U4. (Vin)
- net at U3. (Vin), U4. (Vin): now also U5. (Vin_5V)
- net at M2.1 (PWM): now also U5. (Vin_5V)
- net at C3.1, U1. (Vout): now also U5. (Vin_5V)
- net +BATT: now reaches BT1.1 (+), C1. (-)
- net +BATT: now also C2. (-), M2.2 (+), U1. (Vout), U2. (Vs)
- new net: U3. (Vin), U4. (Vin), U5. (Vin_5V) (x4)
- new net: U2. (Vs), U5. (Vin_5V) (x4)
Other:
- moved on the sheet: M1, U1

Commit message: main_v1.2 schematic
Connections:
- net at U5. (Vin_5V): now also U2. (Vs)
- new net: U3. (Vin), U4. (Vin), U5. (Vin_5V) (x4)
- new net: C3.1, U1. (Vout), U5. (Vin_5V)
- new net: U2. (Vs), U5. (Vin_5V) (x3)
Other:
- moved on the sheet: BT1, C1, C2, C3, M1, M2, U1, U2, U3, U4, U5

Commit message: Created v1-3, added kill switch
Parts:
- added SW1: SW_SPST, symbol Switch:SW_SPST
- U5: value BBB_Wireless_Reduced -> BBB_Wireless
Connections:
- net +BATT: now also SW1.2 (B); no longer BT1.1 (+), C1. (-), C2. (-)
- net at U5. (Vin_5V): now also U2. (Vs)
- new net: U3. (Vin), U4. (Vin), U5. (Vin_5V) (x4)
- new net: C3.1, U1. (Vout), U5. (Vin_5V)
- new net: BT1.1 (+), C1. (-), C2. (-), SW1.1 (A)
- new net: U2. (Vs), U5. (Vin_5V) (x3)
Other:
- moved on the sheet: BT1, C1, C2
Changed lines of the file:
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@@
     (title "Payload Main Circuit")
     (date "2022-12-16")
-    (rev "1.2")
+    (rev "1.3")
   )
   (junction (at 160.02 142.24) (diameter 0) (color 0 0 0 0)
@@
   (junction (at 180.34 43.18) (diameter 0) (color 0 0 0 0)
   )
-  (junction (at 128.27 36.83) (diameter 0) (color 0 0 0 0)
-  )
-  (junction (at 128.27 43.18) (diameter 0) (color 0 0 0 0)
+  (junction (at 132.08 36.83) (diameter 0) (color 0 0 0 0)
+  )
+  (junction (at 113.03 43.18) (diameter 0) (color 0 0 0 0)
   )
   (junction (at 152.4 134.62) (diameter 0) (color 0 0 0 0)
@@
   (junction (at 162.56 144.78) (diameter 0) (color 0 0 0 0)
   )
-  (junction (at 73.66 43.18) (diameter 0) (color 0 0 0 0)
-  )
-  (junction (at 132.08 36.83) (diameter 0) (color 0 0 0 0)
-  )
-  (junction (at 73.66 36.83) (diameter 0) (color 0 0 0 0)
+  (junction (at 58.42 43.18) (diameter 0) (color 0 0 0 0)
+  )
+  (junction (at 113.03 36.83) (diameter 0) (color 0 0 0 0)
+  )
+  (junction (at 58.42 36.83) (diameter 0) (color 0 0 0 0)
   )
   (wire (pts (xy 152.4 134.62) (xy 152.4 160.02))
@@
     (stroke (width 0) (type default) (color 0 0 0 0))
   )
-  (wire (pts (xy 66.04 45.72) (xy 41.91 45.72))
+  (wire (pts (xy 50.8 45.72) (xy 26.67 45.72))
     (stroke (width 0) (type default) (color 0 0 0 0))
   )
@@
     (stroke (width 0) (type default) (color 0 0 0 0))
   )
-  (wire (pts (xy 66.04 34.29) (xy 66.04 36.83))
+  (wire (pts (xy 50.8 34.29) (xy 50.8 36.83))
     (stroke (width 0) (type default) (color 0 0 0 0))
   )
@@
     (stroke (width 0) (type default) (color 0 0 0 0))
   )
-  (wire (pts (xy 66.04 43.18) (xy 66.04 45.72))
+  (wire (pts (xy 50.8 43.18) (xy 50.8 45.72))
     (stroke (width 0) (type default) (color 0 0 0 0))
   )
@@
     (stroke (width 0) (type default) (color 0 0 0 0))
   )
-  (wire (pts (xy 41.91 34.29) (xy 66.04 34.29))
-    (stroke (width 0) (type default) (color 0 0 0 0))
-  )
-  (wire (pts (xy 73.66 43.18) (xy 128.27 43.18))
+  (wire (pts (xy 26.67 34.29) (xy 50.8 34.29))
+    (stroke (width 0) (type default) (color 0 0 0 0))
+  )
+  (wire (pts (xy 58.42 43.18) (xy 113.03 43.18))
     (stroke (width 0) (type default) (color 0 0 0 0))
   )
@@
     (stroke (width 0) (type default) (color 0 0 0 0))
   )
+  (wire (pts (xy 125.73 36.83) (xy 132.08 36.83))
+    (stroke (width 0) (type default) (color 0 0 0 0))
+  )
   (wire (pts (xy 133.35 85.09) (xy 139.7 85.09))
     (stroke (width 0) (type default) (color 0 0 0 0))
@@
     (stroke (width 0) (type default) (color 0 0 0 0))
   )
-  (wire (pts (xy 73.66 36.83) (xy 128.27 36.83))
+  (wire (pts (xy 58.42 36.83) (xy 113.03 36.83))
     (stroke (width 0) (type default) (color 0 0 0 0))
   )
@@
     (stroke (width 0) (type default) (color 0 0 0 0))
   )
-  (wire (pts (xy 128.27 43.18) (xy 132.08 43.18))
+  (wire (pts (xy 113.03 43.18) (xy 132.08 43.18))
     (stroke (width 0) (type default) (color 0 0 0 0))
   )
@@
     (stroke (width 0) (type default) (color 0 0 0 0))
   )
-  (wire (pts (xy 66.04 43.18) (xy 73.66 43.18))
+  (wire (pts (xy 50.8 43.18) (xy 58.42 43.18))
     (stroke (width 0) (type default) (color 0 0 0 0))
   )
@@
     (stroke (width 0) (type default) (color 0 0 0 0))
   )
-  (wire (pts (xy 128.27 36.83) (xy 132.08 36.83))
-    (stroke (width 0) (type default) (color 0 0 0 0))
-  )
-  (wire (pts (xy 66.04 36.83) (xy 73.66 36.83))
+  (wire (pts (xy 50.8 36.83) (xy 58.42 36.83))
     (stroke (width 0) (type default) (color 0 0 0 0))
   )
@@
     (stroke (width 0) (type default) (color 0 0 0 0))
   )
-  (wire (pts (xy 41.91 45.72) (xy 41.91 44.45))
+  (wire (pts (xy 26.67 45.72) (xy 26.67 44.45))
+    (stroke (width 0) (type default) (color 0 0 0 0))
+  )
+  (wire (pts (xy 113.03 36.83) (xy 115.57 36.83))
     (stroke (width 0) (type default) (color 0 0 0 0))
   )
@@
     (pin "")
   )
-  (symbol (lib_id "payload_symbol_library:XT60M") (at 110.49 31.75 0) (unit 1)
+  (symbol (lib_id "payload_symbol_library:XT60M") (at 95.25 31.75 0) (unit 1)
     (in_bom yes) (on_board yes)
-    (property "Reference" "C2" (id 0) (at 116.205 29.21 0))
-    (property "Value" "XT60M" (id 1) (at 116.84 31.75 0))
-    (property "Footprint" "" (id 2) (at 110.49 31.75 0)
-      (effects (font (size 1.27 1.27)) hide)
-    )
-    (property "Datasheet" "" (id 3) (at 110.49 31.75 0)
+    (property "Reference" "C2" (id 0) (at 100.965 29.21 0))
+    (property "Value" "XT60M" (id 1) (at 101.6 31.75 0))
+    (property "Footprint" "" (id 2) (at 95.25 31.75 0)
+      (effects (font (size 1.27 1.27)) hide)
+    )
+    (property "Datasheet" "" (id 3) (at 95.25 31.75 0)
       (effects (font (size 1.27 1.27)) hide)
     )
@@
     (pin "1")
   )
-  (symbol (lib_id "payload_symbol_library:XT60F") (at 95.25 33.02 0) (mirror y) (unit 1)
+  (symbol (lib_id "payload_symbol_library:XT60F") (at 80.01 33.02 0) (mirror y) (unit 1)
     (in_bom yes) (on_board yes)
-    (property "Reference" "C1" (id 0) (at 83.82 29.21 0)
+    (property "Reference" "C1" (id 0) (at 68.58 29.21 0)
       (effects (font (size 1.27 1.27)) (justify right))
     )
-    (property "Value" "XT60F" (id 1) (at 82.55 31.75 0)
+    (property "Value" "XT60F" (id 1) (at 67.31 31.75 0)
       (effects (font (size 1.27 1.27)) (justify right))
     )
-    (property "Footprint" "" (id 2) (at 95.25 33.02 0)
-      (effects (font (size 1.27 1.27)) hide)
-    )
-    (property "Datasheet" "" (id 3) (at 95.25 33.02 0)
+    (property "Footprint" "" (id 2) (at 80.01 33.02 0)
+      (effects (font (size 1.27 1.27)) hide)
+    )
+    (property "Datasheet" "" (id 3) (at 80.01 33.02 0)
       (effects (font (size 1.27 1.27)) hide)
     )
@@
       (effects (font (size 1.27 1.27)) (justify left))
     )
-    (property "Value" "BBB_Wireless_Reduced" (id 1) (at 201.93 94.6149 0)
+    (property "Value" "BBB_Wireless" (id 1) (at 201.93 94.6149 0)
       (effects (font (size 1.27 1.27)) (justify left))
     )
@@
     (pin "2")
   )
+  (symbol (lib_id "Switch:SW_SPST") (at 120.65 36.83 0) (unit 1)
+    (in_bom yes) (on_board yes) (fields_autoplaced)
+    (property "Reference" "SW1" (id 0) (at 120.65 30.48 0))
+    (property "Value" "SW_SPST" (id 1) (at 120.65 33.02 0))
+    (property "Footprint" "" (id 2) (at 120.65 36.83 0)
+      (effects (font (size 1.27 1.27)) hide)
+    )
+    (property "Datasheet" "~" (id 3) (at 120.65 36.83 0)
+      (effects (font (size 1.27 1.27)) hide)
+    )
+    (pin "1")
+    (pin "2")
+  )
   (symbol (lib_id "power:+BATT") (at 144.78 116.84 0) (unit 1)
     (in_bom yes) (on_board yes)
@@
     (pin "1")
   )
-  (symbol (lib_id "Device:Battery") (at 41.91 39.37 0) (unit 1)
-    (in_bom yes) (on_board yes) (fields_autoplaced)
-    (property "Reference" "BT1" (id 0) (at 45.72 37.7189 0)
-      (effects (font (size 1.27 1.27)) (justify left))
-    )
-    (property "Value" "7.4 V 2S LiPo" (id 1) (at 45.72 40.2589 0)
-      (effects (font (size 1.27 1.27)) (justify left))
-    )
-    (property "Footprint" "" (id 2) (at 41.91 37.846 90)
-      (effects (font (size 1.27 1.27)) hide)
-    )
-    (property "Datasheet" "~" (id 3) (at 41.91 37.846 90)
+  (symbol (lib_id "Device:Battery") (at 26.67 39.37 0) (unit 1)
+    (in_bom yes) (on_board yes) (fields_autoplaced)
+    (property "Reference" "BT1" (id 0) (at 30.48 37.7189 0)
+      (effects (font (size 1.27 1.27)) (justify left))
+    )
+    (property "Value" "7.4 V 2S LiPo" (id 1) (at 30.48 40.2589 0)
+      (effects (font (size 1.27 1.27)) (justify left))
+    )
+    (property "Footprint" "" (id 2) (at 26.67 37.846 90)
+      (effects (font (size 1.27 1.27)) hide)
+    )
+    (property "Datasheet" "~" (id 3) (at 26.67 37.846 90)
       (effects (font (size 1.27 1.27)) hide)
     )
@@
       (reference "M2") (unit 1) (value "Motor_Servo") (footprint "")
     )
+    (path "/e73ec205-4335-431a-bc86-dab5f72536c8"
+      (reference "SW1") (unit 1) (value "SW_SPST") (footprint "")
+    )
     (path "/393cc4ab-c0f2-4ff8-bc16-2d8d35b1709f"
       (reference "U1") (unit 1) (value "S13V10FS") (footprint "")
@@
     )
     (path "/6360e655-7c4a-4696-ac85-77737dd12c5a"
-      (reference "U5") (unit 1) (value "BBB_Wireless_Reduced") (footprint "")
-    )
-  )
+      (reference "U5") (unit 1) (value "BBB_Wireless") (footprint "")
+    )
+  )
