File: kicad/cape/cape.kicad_sch (KiCad schematic)
At the start: 6 parts, among them M1 HSR-2648CR, P1 BeagleBone_Black_Header, P2 BeagleBone_Black_Header, SW1 L101011_SPST

Commit message: first working revision of cape done
Parts:
- added R1, R2: 5.6K, Resistor_THT:R_Axial_DIN0207_L6.3mm_D2.5mm_P10.16mm_Horizontal, symbol Device:R
- added U1: L298, Connector_PinSocket_2.54mm:PinSocket_1x06_P2.54mm_Vertical, symbol payload_symbol_library:L298
- added U2: BNO055, Connector_PinSocket_2.54mm:PinSocket_1x06_P2.54mm_Vertical, symbol payload_symbol_library:BNO055
- added U3: BMP390, Connector_PinSocket_2.54mm:PinSocket_1x08_P2.54mm_Vertical, symbol payload_symbol_library:BMP390
- added U4: S13V10FS, Connector_PinSocket_2.54mm:PinSocket_1x03_P2.54mm_Vertical, symbol payload_symbol_library:S13V10FS
Connections:
- net +3.3V: now also R1.1, R2.1, U2.1 (Vin), U3.1 (Vin)
- net +5V: now also U4.3 (Vout); no longer M1.2 (+), SW1.2 (B)
- net GNDD: now also U1.6 (GND), U2.3 (GND), U3.3 (GND), U4.2 (GND)
- net GPIO[117]: now also U1.2 (In_A2)
- net GPIO[122]: now also U1.4 (In_B2)
- net GPIO[125]: now also U1.3 (In_B1)
- net GPIO[20]: now also U2.6 (RST)
- net GPIO[40]: no longer M1.1 (PWM)
- net GPIO[49]: now also U1.1 (In_A1)
- net GPIO[7]: now also M1.1 (PWM)
- net I2C2.SCL: now also R1.2, U2.5 (SCL), U3.4 (SCL)
- net I2C2.SDA: now also R2.2, U2.4 (SDA), U3.6 (SDA)
- net +7.4V: now reaches BT1.1 (+), SW1.1 (A)
- net +7.4V: now also M1.2 (+), U1.5 (Vs)
- new net: SW1.2 (B), U4.1 (Vin)
Other:
- moved on the sheet: BT1, C1
