File: kicad/cape/_autosave-cape.kicad_sch (KiCad schematic)
At the start: 13 parts, among them M1 HSR-2648CR, P1 BeagleBone_Black_Header, P2 BeagleBone_Black_Header, SW1 L101011_SPST, U1 L298, U2 BNO055, U3 BMP390, U4 S13V10FS

Commit message: Finished second revision of cape, basically print-ready
Parts:
- U1: footprint Connector_PinSocket_2.54mm:PinSocket_1x06_P2.54mm_Vertical -> Connector_PinHeader_2.54mm:PinHeader_1x06_P2.54mm_Vertical
Changed lines of the file:
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@@
     (property "Reference" "U1" (id 0) (at 66.04 124.46 0))
     (property "Value" "L298" (id 1) (at 66.04 127 0))
-    (property "Footprint" "Connector_PinSocket_2.54mm:PinSocket_1x06_P2.54mm_Vertical" (id 2) (at 55.88 129.54 0)
+    (property "Footprint" "Connector_PinHeader_2.54mm:PinHeader_1x06_P2.54mm_Vertical" (id 2) (at 55.88 129.54 0)
       (effects (font (size 1.27 1.27)) hide)
     )
@@
     )
     (path "/ecf7c526-1bd5-49c8-a82a-8acc85e22ee0"
-      (reference "U1") (unit 1) (value "L298") (footprint "Connector_PinSocket_2.54mm:PinSocket_1x06_P2.54mm_Vertical")
+      (reference "U1") (unit 1) (value "L298") (footprint "Connector_PinHeader_2.54mm:PinHeader_1x06_P2.54mm_Vertical")
     )
     (path "/ae4a70ec-7099-49d5-8f39-6daa3b0242a8"
