File: kicad/cape/cape.kicad_pcb (KiCad board)
At the start: 2 copper layers, 86.4 x 54.6 mm, 17 parts, among them M1 HSR-2648CR, P1 BeagleBone_Black_Header, P2 BeagleBone_Black_Header, SW1 L101011_SPST, U1 S13V10F5, U2 BNO055, U3 A4988

Commit message: Updated all schematics
Parts:
- removed SW1: L101011_SPST, payload_footprint_library:SW_L101011MS02Q
- added JP1: Jumper_3_Open, Connector_PinHeader_2.54mm:PinHeader_1x03_P2.54mm_Vertical, F.Cu at (70.8, 72.1)
- added U3: stepper_breakout, Connector_PinSocket_2.54mm:PinSocket_1x04_P2.54mm_Vertical, F.Cu at (92.4, 51.7)
- moved BT1 2.88 mm to (65.7, 81.0)
- renumbered U2 to U1, U1 to U2, U3 to U4
Connections:
- U4 pad 3: unconnected-(U3-Pad3) -> Net-(U3-Pad1)
- U4 pad 4: unconnected-(U3-Pad4) -> Net-(U3-Pad2)
- U4 pad 5: unconnected-(U3-Pad5) -> Net-(U3-Pad3)
- U4 pad 6: unconnected-(U3-Pad6) -> Net-(U3-Pad4)
Routing:
- net /+7.4V: track 65.7 -> 56.5 mm
- net Net-(U3-Pad4): track 0.00 -> 5.51 mm
- net Net-(U3-Pad3): track 0.00 -> 5.51 mm
- net Net-(U3-Pad2): track 0.00 -> 5.51 mm
- net Net-(U3-Pad1): track 0.00 -> 5.51 mm
- net Net-(BT1-Pad1): track 10.3 -> 12.0 mm
Other:
- board text added: "1A"
- board text added: "1B"
- board text added: "2A"
- board text added: "2B"
- board text added: "3.3V"
- board text added: "5V"
- board text added: "7.4V"
- board text added: "GND"
- board text added: "Off"
- board text added: "On"
- board text added: "PWM"
