File: kicad/main/main.kicad_sch (KiCad schematic)
At the start: 13 parts, among them J1 XT60F, J2 XT60M, M1 NEMA 8 Bipolar Stepper, M2 HSR-2648CR, SW1 L101011_SPST, U1 A4988, U2 S13V10FS, U3 BeagleBone Black Wireless, U4 BNO055

Commit message: Cape 1.3, Main 1.7
Parts:
- removed U2: S13V10FS, symbol payload_symbol_library:S13V10FS
- added C2: 10 nF, symbol Device:C_Small
- added C3: 100 uF, symbol Device:C_Small
- added U2: S13V10F5, symbol payload_symbol_library:S13V10F5
Connections:
- net +3.3V: now also U3.P9_4 (VDD_3.3V); no longer U3.P9_3 (VDD_3.3V)
- net +BATT: now also U2.1 (Vin)
- net GND: now also C2.2, C3.2, U2.2 (GND)
- net at U3.P9_6 (VDD_5V): now also C2.1, C3.1, U2.3 (Vout)
- net at U4.6 (RST): now also U3.P9_25 (GPIO_117); no longer U3.P9_12 (GPIO_60)
- net at U4.9 (INT): now also U3.P9_30 (GPIO_112); no longer U3.P9_15 (GPIO_48)
- net at U1.13 (~{RESET}): now also U3.P8_15 (GPIO_47); no longer U3.P9_23 (GPIO_49)
- net at U1.14 (~{SLEEP}): now also U3.P8_17 (GPIO_27); no longer U3.P9_25 (GPIO_117)
- net at U1.15 (STEP): now also U3.P8_18 (GPIO_65); no longer U3.P9_27 (GPIO_115)
- net at U1.16 (DIR): now also U3.P8_26 (GPIO_61); no longer U3.P9_30 (GPIO_112)
Changed lines of the file:
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@@
   (title_block
     (title "Payload Main Subsystem")
-    (date "2022-12-29")
-    (rev "1.6")
+    (date "2022-12-30")
+    (rev "1.7")
   )
   (junction (at 95.25 27.94) (diameter 0) (color 0 0 0 0)
@@
   (junction (at 104.14 33.02) (diameter 0) (color 0 0 0 0)
   )
+  (junction (at 132.08 24.13) (diameter 0) (color 0 0 0 0)
+  )
   (junction (at 162.56 52.07) (diameter 0) (color 0 0 0 0)
   )
@@
   (junction (at 87.63 24.13) (diameter 0) (color 0 0 0 0)
   )
+  (junction (at 137.16 24.13) (diameter 0) (color 0 0 0 0)
+  )
   (junction (at 95.25 24.13) (diameter 0) (color 0 0 0 0)
   )
   (junction (at 95.25 33.02) (diameter 0) (color 0 0 0 0)
+  )
+  (junction (at 144.78 29.21) (diameter 0) (color 0 0 0 0)
   )
   (no_connect (at 191.77 64.77))
@@
     (stroke (width 0) (type default) (color 0 0 0 0))
   )
+  (wire (pts (xy 144.78 29.21) (xy 149.86 29.21))
+    (stroke (width 0) (type default) (color 0 0 0 0))
+  )
   (wire (pts (xy 95.25 35.56) (xy 95.25 33.02))
     (stroke (width 0) (type default) (color 0 0 0 0))
   )
+  (wire (pts (xy 132.08 24.13) (xy 137.16 24.13))
+    (stroke (width 0) (type default) (color 0 0 0 0))
+  )
   (wire (pts (xy 158.75 64.77) (xy 162.56 64.77))
     (stroke (width 0) (type default) (color 0 0 0 0))
@@
     (stroke (width 0) (type default) (color 0 0 0 0))
   )
+  (wire (pts (xy 144.78 29.21) (xy 144.78 31.75))
+    (stroke (width 0) (type default) (color 0 0 0 0))
+  )
   (wire (pts (xy 158.75 62.23) (xy 160.02 62.23))
     (stroke (width 0) (type default) (color 0 0 0 0))
@@
     (stroke (width 0) (type default) (color 0 0 0 0))
   )
+  (wire (pts (xy 137.16 29.21) (xy 144.78 29.21))
+    (stroke (width 0) (type default) (color 0 0 0 0))
+  )
   (wire (pts (xy 106.68 67.31) (xy 106.68 62.23))
     (stroke (width 0) (type default) (color 0 0 0 0))
@@
   )
   (wire (pts (xy 88.9 62.23) (xy 106.68 62.23))
+    (stroke (width 0) (type default) (color 0 0 0 0))
+  )
+  (wire (pts (xy 137.16 24.13) (xy 149.86 24.13))
     (stroke (width 0) (type default) (color 0 0 0 0))
   )
@@
     (pin "1")
   )
+  (symbol (lib_id "Device:C_Small") (at 137.16 26.67 0) (unit 1)
+    (in_bom yes) (on_board yes) (fields_autoplaced)
+    (property "Reference" "C2" (id 0) (at 139.7 25.4062 0)
+      (effects (font (size 1.27 1.27)) (justify left))
+    )
+    (property "Value" "10 nF" (id 1) (at 139.7 27.9462 0)
+      (effects (font (size 1.27 1.27)) (justify left))
+    )
+    (property "Footprint" "" (id 2) (at 137.16 26.67 0)
+      (effects (font (size 1.27 1.27)) hide)
+    )
+    (property "Datasheet" "~" (id 3) (at 137.16 26.67 0)
+      (effects (font (size 1.27 1.27)) hide)
+    )
+    (pin "1")
+    (pin "2")
+  )
   (symbol (lib_id "Motor:Motor_Servo") (at 92.71 91.44 0) (mirror y) (unit 1)
     (in_bom yes) (on_board yes)
@@
     (pin "1")
   )
-  (symbol (lib_id "payload_symbol_library:S13V10FS") (at 123.19 21.59 0) (unit 1)
-    (in_bom yes) (on_board yes) (fields_autoplaced)
-    (property "Reference" "U2" (id 0) (at 115.57 16.51 0))
-    (property "Value" "S13V10FS" (id 1) (at 115.57 19.05 0))
-    (property "Footprint" "" (id 2) (at 123.19 21.59 0)
-      (effects (font (size 1.27 1.27)) hide)
-    )
-    (property "Datasheet" "" (id 3) (at 123.19 21.59 0)
-      (effects (font (size 1.27 1.27)) hide)
-    )
-    (pin "1")
-    (pin "2")
-    (pin "3")
-  )
   (symbol (lib_id "payload_symbol_library:XT60M") (at 59.69 22.86 0) (unit 1)
     (in_bom yes) (on_board yes)
@@
     )
     (pin "P8_13")
-    (pin "P9_12")
-    (pin "P9_15")
+    (pin "P8_15")
+    (pin "P8_17")
+    (pin "P8_18")
+    (pin "P8_26")
     (pin "P9_19")
     (pin "P9_2")
     (pin "P9_20")
-    (pin "P9_23")
     (pin "P9_25")
-    (pin "P9_27")
-    (pin "P9_3")
     (pin "P9_30")
+    (pin "P9_4")
     (pin "P9_6")
   )
+  (symbol (lib_id "payload_symbol_library:S13V10F5") (at 123.19 21.59 0) (unit 1)
+    (in_bom yes) (on_board yes) (fields_autoplaced)
+    (property "Reference" "U2" (id 0) (at 115.57 16.51 0))
+    (property "Value" "S13V10F5" (id 1) (at 115.57 19.05 0))
+    (property "Footprint" "" (id 2) (at 123.19 21.59 0)
+      (effects (font (size 1.27 1.27)) hide)
+    )
+    (property "Datasheet" "" (id 3) (at 123.19 21.59 0)
+      (effects (font (size 1.27 1.27)) hide)
+    )
+    (pin "1")
+    (pin "2")
+    (pin "3")
+  )
   (symbol (lib_id "Device:R") (at 162.56 57.15 0) (unit 1)
     (in_bom yes) (on_board yes)
@@
     )
     (property "Datasheet" "~" (id 3) (at 162.56 57.15 0)
+      (effects (font (size 1.27 1.27)) hide)
+    )
+    (pin "1")
+    (pin "2")
+  )
+  (symbol (lib_id "Device:C_Small") (at 149.86 26.67 0) (unit 1)
+    (in_bom yes) (on_board yes) (fields_autoplaced)
+    (property "Reference" "C3" (id 0) (at 152.4 25.4062 0)
+      (effects (font (size 1.27 1.27)) (justify left))
+    )
+    (property "Value" "100 uF" (id 1) (at 152.4 27.9462 0)
+      (effects (font (size 1.27 1.27)) (justify left))
+    )
+    (property "Footprint" "" (id 2) (at 149.86 26.67 0)
+      (effects (font (size 1.27 1.27)) hide)
+    )
+    (property "Datasheet" "~" (id 3) (at 149.86 26.67 0)
       (effects (font (size 1.27 1.27)) hide)
     )
@@
     )
     (property "Datasheet" "" (id 3) (at 57.15 50.8 0)
+      (effects (font (size 1.27 1.27)) hide)
+    )
+    (pin "1")
+  )
+  (symbol (lib_id "power:GND") (at 144.78 31.75 0) (unit 1)
+    (in_bom yes) (on_board yes) (fields_autoplaced)
+    (property "Reference" "#PWR09" (id 0) (at 144.78 38.1 0)
+      (effects (font (size 1.27 1.27)) hide)
+    )
+    (property "Value" "GND" (id 1) (at 144.78 36.83 0))
+    (property "Footprint" "" (id 2) (at 144.78 31.75 0)
+      (effects (font (size 1.27 1.27)) hide)
+    )
+    (property "Datasheet" "" (id 3) (at 144.78 31.75 0)
       (effects (font (size 1.27 1.27)) hide)
     )
@@
       (reference "#PWR08") (unit 1) (value "GND") (footprint "")
     )
+    (path "/9d1c4416-be2b-4534-959b-8aaef2b0de36"
+      (reference "#PWR09") (unit 1) (value "GND") (footprint "")
+    )
     (path "/ec287280-009c-4228-95d6-4a5138809f2b"
       (reference "BT1") (unit 1) (value "7.4 V 2S LiPo") (footprint "")
@@
       (reference "C1") (unit 1) (value "100 uF") (footprint "")
     )
+    (path "/21fd3ae7-6422-408e-b04d-ba114fb3f286"
+      (reference "C2") (unit 1) (value "10 nF") (footprint "")
+    )
+    (path "/890ead54-64e2-49d4-bbac-7e664de4dcaf"
+      (reference "C3") (unit 1) (value "100 uF") (footprint "")
+    )
     (path "/4d09686c-8870-440a-9631-39a3bc7b1f60"
       (reference "J1") (unit 1) (value "XT60F") (footprint "")
@@
       (reference "U1") (unit 1) (value "A4988") (footprint "Module:Pololu_Breakout-16_15.2x20.3mm")
     )
-    (path "/393cc4ab-c0f2-4ff8-bc16-2d8d35b1709f"
-      (reference "U2") (unit 1) (value "S13V10FS") (footprint "")
+    (path "/76683f8f-ede7-454d-8678-18abf3b4592c"
+      (reference "U2") (unit 1) (value "S13V10F5") (footprint "")
     )
     (path "/6360e655-7c4a-4696-ac85-77737dd12c5a"

Commit message: Updated all schematics
Parts:
- removed SW1: L101011_SPST, symbol Switch:SW_SPST
- added JP1: Jumper_3_Open, symbol Jumper:Jumper_3_Open
Connections:
- net +BATT: now also JP1.3 (B)
- new net: J2. (-), JP1.2 (C)
- no-connect marks 8 -> 9
Other:
- company: (none) -> Peter Costescu
Changed lines of the file:
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@@
     (title "Payload Main Subsystem")
     (date "2022-12-30")
-    (rev "1.7")
+    (rev "1.8")
+    (company "Peter Costescu")
   )
   (junction (at 95.25 27.94) (diameter 0) (color 0 0 0 0)
@@
   (junction (at 162.56 52.07) (diameter 0) (color 0 0 0 0)
   )
+  (junction (at 87.63 24.13) (diameter 0) (color 0 0 0 0)
+  )
   (junction (at 73.66 83.82) (diameter 0) (color 0 0 0 0)
   )
@@
   )
   (junction (at 167.64 67.31) (diameter 0) (color 0 0 0 0)
-  )
-  (junction (at 87.63 24.13) (diameter 0) (color 0 0 0 0)
   )
   (junction (at 137.16 24.13) (diameter 0) (color 0 0 0 0)
@@
   (no_connect (at 88.9 69.85))
   (no_connect (at 88.9 74.93))
+  (no_connect (at 67.31 20.32))
   (no_connect (at 191.77 69.85))
   (no_connect (at 88.9 59.69))
@@
     (stroke (width 0) (type default) (color 0 0 0 0))
   )
+  (wire (pts (xy 83.82 24.13) (xy 87.63 24.13))
+    (stroke (width 0) (type default) (color 0 0 0 0))
+  )
   (wire (pts (xy 114.3 73.66) (xy 114.3 88.9))
     (stroke (width 0) (type default) (color 0 0 0 0))
@@
     (stroke (width 0) (type default) (color 0 0 0 0))
   )
+  (wire (pts (xy 83.82 20.32) (xy 83.82 24.13))
+    (stroke (width 0) (type default) (color 0 0 0 0))
+  )
   (wire (pts (xy 109.22 64.77) (xy 116.84 64.77))
     (stroke (width 0) (type default) (color 0 0 0 0))
@@
     (stroke (width 0) (type default) (color 0 0 0 0))
   )
-  (wire (pts (xy 80.01 24.13) (xy 87.63 24.13))
-    (stroke (width 0) (type default) (color 0 0 0 0))
-  )
   (wire (pts (xy 88.9 64.77) (xy 104.14 64.77))
     (stroke (width 0) (type default) (color 0 0 0 0))
@@
     (stroke (width 0) (type default) (color 0 0 0 0))
   )
-  (wire (pts (xy 66.04 24.13) (xy 69.85 24.13))
-    (stroke (width 0) (type default) (color 0 0 0 0))
-  )
   (wire (pts (xy 160.02 52.07) (xy 162.56 52.07))
     (stroke (width 0) (type default) (color 0 0 0 0))
@@
     (stroke (width 0) (type default) (color 0 0 0 0))
   )
+  (wire (pts (xy 66.04 24.13) (xy 73.66 24.13))
+    (stroke (width 0) (type default) (color 0 0 0 0))
+  )
   (wire (pts (xy 66.04 59.69) (xy 44.45 59.69))
     (stroke (width 0) (type default) (color 0 0 0 0))
   )
+  (wire (pts (xy 80.01 20.32) (xy 83.82 20.32))
+    (stroke (width 0) (type default) (color 0 0 0 0))
+  )
   (wire (pts (xy 49.53 74.93) (xy 55.88 74.93))
     (stroke (width 0) (type default) (color 0 0 0 0))
@@
     (stroke (width 0) (type default) (color 0 0 0 0))
   )
-  (image (at 133.35 111.76)
+  (image (at 143.51 111.76)
     (data
       iVBORw0KGgoAAAANSUhEUgAAAbIAAACKCAYAAADPLc9oAAAABHNCSVQICAgIfAhkiAAAAAlwSFlz
@@
   (symbol (lib_id "power:GND") (at 170.18 76.2 0) (unit 1)
     (in_bom yes) (on_board yes) (fields_autoplaced)
-    (property "Reference" "#PWR08" (id 0) (at 170.18 82.55 0)
+    (property "Reference" "#PWR09" (id 0) (at 170.18 82.55 0)
       (effects (font (size 1.27 1.27)) hide)
     )
@@
   (symbol (lib_id "payload_symbol_library:XT60M") (at 59.69 22.86 0) (unit 1)
     (in_bom yes) (on_board yes)
-    (property "Reference" "J2" (id 0) (at 62.865 17.78 0))
-    (property "Value" "XT60M" (id 1) (at 63.5 20.32 0))
+    (property "Reference" "J2" (id 0) (at 61.595 30.48 0))
+    (property "Value" "XT60M" (id 1) (at 62.23 33.02 0))
     (property "Footprint" "" (id 2) (at 59.69 22.86 0)
       (effects (font (size 1.27 1.27)) hide)
@@
   (symbol (lib_id "payload_symbol_library:XT60F") (at 57.15 24.13 0) (mirror y) (unit 1)
     (in_bom yes) (on_board yes)
-    (property "Reference" "J1" (id 0) (at 53.34 17.78 0)
+    (property "Reference" "J1" (id 0) (at 52.07 30.48 0)
       (effects (font (size 1.27 1.27)) (justify right))
     )
-    (property "Value" "XT60F" (id 1) (at 52.07 20.32 0)
+    (property "Value" "XT60F" (id 1) (at 50.8 33.02 0)
       (effects (font (size 1.27 1.27)) (justify right))
     )
@@
   )
   (symbol (lib_id "power:PWR_FLAG") (at 87.63 24.13 0) (unit 1)
-    (in_bom yes) (on_board yes) (fields_autoplaced)
+    (in_bom yes) (on_board yes)
     (property "Reference" "#FLG01" (id 0) (at 87.63 22.225 0)
       (effects (font (size 1.27 1.27)) hide)
     )
-    (property "Value" "PWR_FLAG" (id 1) (at 87.63 19.05 0))
+    (property "Value" "PWR_FLAG" (id 1) (at 88.9 20.32 0))
     (property "Footprint" "" (id 2) (at 87.63 24.13 0)
       (effects (font (size 1.27 1.27)) hide)
@@
     (pin "1")
   )
+  (symbol (lib_id "Jumper:Jumper_3_Open") (at 73.66 20.32 0) (unit 1)
+    (in_bom yes) (on_board yes) (fields_autoplaced)
+    (property "Reference" "JP1" (id 0) (at 73.66 13.97 0))
+    (property "Value" "Jumper_3_Open" (id 1) (at 73.66 16.51 0))
+    (property "Footprint" "" (id 2) (at 73.66 20.32 0)
+      (effects (font (size 1.27 1.27)) hide)
+    )
+    (property "Datasheet" "~" (id 3) (at 73.66 20.32 0)
+      (effects (font (size 1.27 1.27)) hide)
+    )
+    (pin "1")
+    (pin "2")
+    (pin "3")
+  )
   (symbol (lib_id "power:GND") (at 144.78 31.75 0) (unit 1)
     (in_bom yes) (on_board yes) (fields_autoplaced)
-    (property "Reference" "#PWR09" (id 0) (at 144.78 38.1 0)
+    (property "Reference" "#PWR08" (id 0) (at 144.78 38.1 0)
       (effects (font (size 1.27 1.27)) hide)
     )
@@
     (pin "2")
   )
-  (symbol (lib_id "Switch:SW_SPST") (at 74.93 24.13 0) (unit 1)
-    (in_bom yes) (on_board yes) (fields_autoplaced)
-    (property "Reference" "SW1" (id 0) (at 74.93 17.78 0))
-    (property "Value" "L101011_SPST" (id 1) (at 74.93 20.32 0))
-    (property "Footprint" "" (id 2) (at 74.93 24.13 0)
-      (effects (font (size 1.27 1.27)) hide)
-    )
-    (property "Datasheet" "~" (id 3) (at 74.93 24.13 0)
-      (effects (font (size 1.27 1.27)) hide)
-    )
-    (pin "1")
-    (pin "2")
-  )
   (symbol (lib_id "power:+BATT") (at 128.27 90.17 0) (unit 1)
     (in_bom yes) (on_board yes)
@@
       (reference "#PWR07") (unit 1) (value "+BATT") (footprint "")
     )
+    (path "/9d1c4416-be2b-4534-959b-8aaef2b0de36"
+      (reference "#PWR08") (unit 1) (value "GND") (footprint "")
+    )
     (path "/37de6bbb-6273-4906-807b-25c12386cb60"
-      (reference "#PWR08") (unit 1) (value "GND") (footprint "")
-    )
-    (path "/9d1c4416-be2b-4534-959b-8aaef2b0de36"
       (reference "#PWR09") (unit 1) (value "GND") (footprint "")
     )
@@
       (reference "J2") (unit 1) (value "XT60M") (footprint "")
     )
+    (path "/9c0488df-4fbe-4ed4-a042-48cd58c8b662"
+      (reference "JP1") (unit 1) (value "Jumper_3_Open") (footprint "")
+    )
     (path "/c539e74f-c9b8-43cc-9641-ae0b6f11b03b"
       (reference "M1") (unit 1) (value "NEMA 8 Bipolar Stepper") (footprint "")
@@
       (reference "R2") (unit 1) (value "5.6K") (footprint "")
     )
-    (path "/e73ec205-4335-431a-bc86-dab5f72536c8"
-      (reference "SW1") (unit 1) (value "L101011_SPST") (footprint "")
-    )
     (path "/b49d0fa0-778f-4fbe-8301-0095ef3304a9"
